Commit message: paper

File: src/pkg/rover_description_pkg/urdf/rover_gazebo.xacro (robot description, xacro)
@@ -114,5 +114,5 @@
     </xacro:sensor_d435i>  -->
     <joint name="camera_to_payload" type="fixed">
-        <origin xyz="0.1 0.0 0.04" rpy="0 0 0"/>
+        <origin xyz="0.15 0.0 0.04" rpy="0 0 0"/>
         <parent link="payload_link"/>
         <child link="${camera_base_frame}"/>
@@ -189,4 +189,5 @@
 			<topic>rover/depth/image_raw</topic>
             <ignition_frame_id>rover/camera_depth_optical_frame</ignition_frame_id>
+            <gz_frame_id>rover/camera_depth_optical_frame</gz_frame_id>
 			<pose>0 0.0 0.0 0 -0 0</pose>
 			<camera name="d435">
@@ -195,6 +196,6 @@
 				<horizontal_fov>1.48702</horizontal_fov>
 				<image>
-					<width>1280</width>
-					<height>720</height>
+					<width>640</width>
+					<height>480</height>
 				</image>
 				<clip>
