Commit message: feat: multi-robot simulation setup
- Added headless mode support to rover_garden.launch.py
- Configured use_sim_time=true for all nodes for proper time synchronization
- Updated world file leonardo_race.sdf with proper plugin configuration
- Modified Docker configuration to use rover_ws workspace
- Enhanced launch file with conditional GUI/headless mode
- Added proper GZ_SIM_RESOURCE_PATH for mesh files access
- Improved rover spawning with transport timeout configuration

File: src/pkg/rover_description_pkg/urdf/rover_macro.xacro (robot description, xacro)
@@ -96,5 +96,7 @@
                 <origin xyz="0 0 0" rpy="-1.57 0.0 3.1415"/>
                 <geometry>
-                    <mesh filename="file://$(find rover_description_pkg)/meshes/rplidar_s2.dae"/>
+                    <!-- TEMP: Cylinder instead of mesh for Docker container compatibility -->
+                    <cylinder radius="0.04" length="0.15"/>
+                    <!-- <mesh filename="file://$(find rover_description_pkg)/meshes/rplidar_s2.dae"/> -->
                 </geometry>
             </visual>
